File: PentagrammicDipyramid/hardware/PentagrammicDipyramid/PentagrammicDipyramid.kicad_pcb (KiCad board)
At the start: 2 copper layers, 22.9 x 97.1 mm, 75 parts

Commit message: RhombicDodecahedron
Parts:
- removed + (x2), G (x2), IN, OUT: Conn_01x01, Connector_PinSocket_2.54mm:PinSocket_1x01_P2.54mm_Vertical
- added ? (x5): , Graphics, F.Cu at (46.0, 10.4)
- added ?: , Graphics, B.Cu at (46.0, 10.4)
- added J1: Conn_01x01, Connector_PinSocket_2.54mm:PinSocket_1x01_P2.54mm_Vertical, F.Cu at (24.0, 38.8)
- added J2: Conn_01x01, Connector_PinSocket_2.54mm:PinSocket_1x01_P2.54mm_Vertical, F.Cu at (23.9, 85.6)
- added J3: Conn_01x01, Connector_PinSocket_2.54mm:PinSocket_1x01_P2.54mm_Vertical, F.Cu at (27.5, 46.5)
- added J4: Conn_01x01, Connector_PinSocket_2.54mm:PinSocket_1x01_P2.54mm_Vertical, F.Cu at (27.7, 78.2)
- added J5: Conn_01x01, Connector_PinSocket_2.54mm:PinSocket_1x01_P2.54mm_Vertical, F.Cu at (32.3, 57.3)
- added J6: Conn_01x01, Connector_PinSocket_2.54mm:PinSocket_1x01_P2.54mm_Vertical, F.Cu at (32.3, 67.1)
- moved H1 0.40 mm to (17.1, 25.8)
- moved ROW2 0.32 mm to (15.8, 65.6)
- moved H3 0.30 mm to (34.2, 62.2)
- moved ROW1 0.28 mm to (19.4, 29.1)
Routing:
- net +5V: track 223.1 -> 231.6 mm, vias 0 -> 2
Other:
- board size 22.9 x 97.1 mm -> 22.9 x 91.8 mm
