File: PentagrammicDipyramid/hardware/PentagrammicDipyramid/PentagrammicDipyramid.kicad_sch (KiCad schematic)
At the start: 69 parts, among them J1 Conn_01x01, J2 Conn_01x01, J3 Conn_01x01, J4 Conn_01x01, J5 Conn_01x01, J6 Conn_01x01

Commit message: RhombicDodecahedron
Other:
- moved on the sheet: LED1, LED10, LED11, LED12, LED13, LED14, LED15, LED16, LED17, LED18, LED19, LED2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
